File: kicad/arduino-focuser/arduino-focuser.kicad_sch (KiCad schematic)
At the start: 2 parts

Commit message: Updating Diagram
Parts:
- added C1: 470uf, symbol Device:C_Polarized_US
- added J1: Conn_01x04, symbol Connector_Generic:Conn_01x04
- added U3: ~, symbol Arduino_Library:SSD1306
Connections:
- net -5V is gone; now on net +5V: U2.10 (VDD), U2.5 (RST), U2.6 (SLP)
- net GND: now also U1.29 (GND), U2.15 (GND), C1.2, U3.1 (GND)
- net at U2.11 (1B): now also J1.4 (Pin_4)
- net at U2.12 (1A): now also J1.3 (Pin_3)
- net at U2.13 (2A): now also J1.2 (Pin_2)
- net at U2.14 (2B): now also J1.1 (Pin_1)
- net +12V: now reaches U2.16 (VMOT)
- net +12V: now also C1.1
- net at U1.23 (SDA/A4/D18): now also U3.4 (SDA)
- net at U1.24 (SCL/A5/D19): now also U3.3 (SCL)
- net +5V: now reaches U1.27 (5V)
- net +5V: now also U3.2 (VCC)
- no-connect marks 0 -> 21
Other:
- note added: "Simple Wiring Diagram"
- note added: "This diagram is not 100% complete, it just shows the wiring of a prototype."
